File: Hardware/CCController/CCController.kicad_pcb (KiCad board)
At the start: 2 copper layers, 180 x 80 mm, 89 parts, among them IC1 CH32V003F4U6, IC2 RY8310, J11 Conn_01x02_Pin, J12 TagConnect, J13 Conn_01x03_Socket, Q1 AO3401A, U1 BP1808, U2 BP1808, U3 BP1808, U4 BP1808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

Commit message: edit Strip controller and buy first batch
Parts:
- added D11: LED_RGB, LED_SMD:LED_RGB_Getian_GT-P6PRGB4303, F.Cu at (117.9, 39.5)
- added D12: LED_RGB, LED_SMD:LED_RGB_Getian_GT-P6PRGB4303, F.Cu at (161.5, 39.6)
- added D13: LED_RGB, LED_SMD:LED_RGB_Getian_GT-P6PRGB4303, F.Cu at (202.8, 39.8)
- moved R2 140.6 mm to (186.8, 45.5), turned to 90 degrees
- moved R4 138.8 mm to (186.9, 60.1), turned to 90 degrees
- moved C8 135.5 mm to (186.9, 38.8), turned to 90 degrees
- moved L2 133.9 mm to (181.7, 44.5), turned to 90 degrees
- moved L4 133.0 mm to (181.7, 59.1), turned to 90 degrees
- moved C7 132.5 mm to (184.4, 38.8), turned to 90 degrees
- moved C16 131.9 mm to (187.0, 53.4), turned to 90 degrees
- moved C6 129.5 mm to (181.9, 38.8), turned to 90 degrees
- moved C15 129.5 mm to (184.5, 53.4), turned to 90 degrees
- moved C14 127.1 mm to (182.0, 53.4), turned to 90 degrees
- moved U4 126.7 mm to (175.0, 58.7), turned to 90 degrees
- moved C5 126.6 mm to (179.4, 38.8), turned to 90 degrees
- moved U2 125.9 mm to (174.9, 44.1), turned to 90 degrees
- moved C13 124.7 mm to (179.5, 53.4), turned to 90 degrees
- moved U1 120.1 mm to (185.0, 22.9), turned to -90 degrees
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Other:
- board size 180 x 80 mm -> 180 x 131.1 mm
