File: Hardware/CCController/CCController.kicad_sch (KiCad schematic)
At the start: 36 parts, among them IC2 CH32V003F4U6, J1 Conn_01x03_Socket, J5 TagConnect, U2 MAX485E, Y1 Crystal_GND23

Commit message: add Files
Parts:
- removed U7, U8, U9: ~, symbol Techbeard:LED_RGBWA
- added J1, J2, J3, J4, J5, J6: Conn_01x01_Socket, symbol Connector:Conn_01x01_Socket
Connections:
- net B+: now also J5.1 (Pin_1)
- net B-: now also J6.1 (Pin_1)
- net G+: now also J3.1 (Pin_1)
- net G-: now also J4.1 (Pin_1)
- net R+: now also J1.1 (Pin_1)
- net R-: now also J2.1 (Pin_1)
Other:
- removed sheet DCDC_CC3
- removed sheet DCDC_CC4
